File: clock_sync.kicad_sch (KiCad schematic)
At the start: 0 parts

Commit message: checkpoint: integrate GNSS RF and ADF4351 reference clock
Parts:
- added C32, C34, C36: 10p, Capacitor_SMD:C_0402_1005Metric, symbol Device:C_Small
- added C33, C35, C37, C39, C41, C43, C45, C47, C50: 100n, Capacitor_SMD:C_0402_1005Metric, symbol Device:C_Small
- added C38, C40, C42, C44, C46, C49: 100p, Capacitor_SMD:C_0402_1005Metric, symbol Device:C_Small
- added C48: 1u, Capacitor_SMD:C_0603_1608Metric, symbol Device:C_Small
- added C51: 1u, Capacitor_SMD:C_0603_1608Metric_Pad1.08x0.95mm_HandSolder, symbol Device:C_Small
- added R28: 5.1k, Resistor_SMD:R_0402_1005Metric, symbol Device:R_Small
- added R29: 10k, Resistor_SMD:R_0402_1005Metric, symbol Device:R_Small
- added R30: 1k, Resistor_SMD:R_0603_1608Metric_Pad0.98x0.95mm_HandSolder, symbol Device:R_Small
- added R31: 120k, Resistor_SMD:R_0603_1608Metric_Pad0.98x0.95mm_HandSolder, symbol Device:R_Small
- added R32: 100k, Resistor_SMD:R_0603_1608Metric_Pad0.98x0.95mm_HandSolder, symbol Device:R_Small
- added R33, R34: 33, Resistor_SMD:R_0603_1608Metric_Pad0.98x0.95mm_HandSolder, symbol Device:R_Small
- added U6: ADF4351, Package_CSP:LFCSP-32-1EP_5x5mm_P0.5mm_EP3.25x3.25mm, symbol Timer_PLL:ADF4351
- added Y1: FVTO10.000M3.3SM5-1.0/1.0C, Crystal:Crystal_SMD_5032-4Pin_5.0x3.2mm, symbol Oscillator:ABLNO
Connections:
- new net: R28.2, U6.22 (RSET)
- new net 3V3_PLL: C38.1, C39.1, C40.1, C41.1, C42.2, C43.2, C44.1, C45.1, C46.1, C47.1, C48.1, C49.1, C50.2, R31.2, U6.10 (AVDD), U6.16 (VVCO), U6.17 (VVCO), U6.28 (DVDD), U6.32 (SDVDD), U6.4 (CE), U6.6 (Vp), Y1.4 (VDD)
- new net ADF_REF_10M: R33.2, R34.2, U6.29 (REFIN)
- new net GND: C32.2, C33.2, C34.2, C35.2, C36.2, C37.2, C38.2, C39.2, C40.2, C41.2, C42.1, C43.1, C44.2, C45.2, C46.2, C47.2, C48.2, C49.2, C50.1, C51.2, R28.1, R29.2, R32.1, U6.11 (AGNDVCO), U6.18 (AGNDVCO), U6.21 (AGNDVCO), U6.27 (DGND), U6.31 (SDGND), U6.33 (EP), U6.8 (CPGND), U6.9 (AGND), Y1.2 (GND)
- new net PLL_LE: U6.3 (LE)
- new net PLL_LOCK: U6.25 (LD)
- new net PLL_RF_EN: R29.1, U6.26 (PDB_RF)
- new net RF_SPI_MOSI: U6.2 (DATA)
- new net RF_SPI_SCK: U6.1 (CLK)
- new net TEMP: C32.1, C33.1, U6.19 (TEMP)
- new net VCOM: C34.1, C35.1, U6.23 (VCOM)
- new net VCTCXO_CTRL: R30.1
- new net VCTCXO_VCTRL: C51.1, R30.2, R31.1, R32.2, Y1.1 (Vctrl)
- new net VREF: C36.1, C37.1, U6.24 (VREF)
