File: gps_l1.kicad_sch (KiCad schematic)
At the start: 0 parts

Commit message: Make schema of dac and rf partly
Parts:
- added C20, C21: 100n, Capacitor_SMD:C_0603_1608Metric, symbol Device:C_Small
- added C22: 10n, Capacitor_SMD:C_0402_1005Metric, symbol Device:C_Small
- added C23: 1u, Capacitor_SMD:C_0603_1608Metric, symbol Device:C_Small
- added C24, C25: 100n, Capacitor_SMD:C_0402_1005Metric, symbol Device:C_Small
- added C26: 10n, Capacitor_SMD:C_0402_1005Metric_Pad0.74x0.62mm_HandSolder, symbol Device:C_Small
- added C27: 6.8p, Capacitor_SMD:C_0603_1608Metric, symbol Device:C_Small
- added L5, L6: 130n, Inductor_SMD:L_0402_1005Metric, symbol Device:L_Small
- added L7, L8: 6.8n, Inductor_SMD:L_0402_1005Metric, symbol Device:L_Small
- added R11: 0, Resistor_SMD:R_0603_1608Metric_Pad0.98x0.95mm_HandSolder, symbol Device:R_Small
- added R12: 4.75k, Resistor_SMD:R_0402_1005Metric_Pad0.72x0.64mm_HandSolder, symbol Device:R_Small
- added R13: 10k, Resistor_SMD:R_0402_1005Metric_Pad0.72x0.64mm_HandSolder, symbol Device:R_Small
- added TR1: TC1-1-13M+, Transformer_SMD:Transformer_MiniCircuits_AT224-1A, symbol Transformer:TC1-1-13M+
- added TR2: BD1222J50200AHF, RF_Converter:Anaren_0805_2012Metric-6, symbol gnss-lib:BD1222J50200AHF
- added U2: LTC5510, Package_DFN_QFN:QFN-16-1EP_4x4mm_P0.65mm_EP2.15x2.15mm, symbol gnss-lib:LTC5510
- added U5: PE4312, gnss_lib:QFN-20-1EP_4x4mm_P0.5mm_EP2.2x2.2mm, symbol gnss-lib:PE4312
Connections:
- new net: L6.1, TR1.3
- new net: C21.1, L6.2
- new net: R11.2, U2.4 (LGND)
- new net: C20.1, L5.2
- new net: L5.1, TR1.1
- new net: C24.1, U2.14 (LO-)
- new net: C25.1, U2.15 (LO+)
- new net: R12.2, U2.8 (I_ADJ)
- new net: L8.1, TR2.4 (BP)
- new net: C27.2, TR2.1 (UP)
- new net: L7.2, TR2.3 (BP)
- new net 5V_MIX: C22.1, C23.1, C26.1, TR2.2 (GND/DC_FEED)
- new net DAC_IF_FILT: TR1.6
- new net GND: C22.2, C23.2, C24.2, C26.2, R11.1, R12.1, R13.1, TR1.4, TR2.5 (GND), U2.12 (GND), U2.13 (GND), U2.16 (TP), U2.17 (EP), U2.9 (GND)
- new net GPS_L1_MIX_OUT: C27.1
- new net LO_MIX: C25.2
- new net LTC5510_IN+: C20.2, U2.2 (IN+)
- new net LTC5510_IN-: C21.2, U2.3 (IN-)
- new net LTC5510_OUT+: L7.1, U2.11 (OUT+)
- new net LTC5510_OUT-: L8.2, U2.10 (OUT-)
- new net MIX_EN: R13.2, U2.5 (EN)
- no-connect marks 0 -> 1

Commit message: checkpoint: integrate GNSS RF and ADF4351 reference clock
Parts:
- added C28, C29: 100p, Capacitor_SMD:C_0603_1608Metric, symbol Device:C_Small
- added C30: 100n, Capacitor_SMD:C_0402_1005Metric_Pad0.74x0.62mm_HandSolder, symbol Device:C_Small
- added C31: 47p, Capacitor_SMD:C_0402_1005Metric, symbol Device:C_Small
- added FL1: SAFEB1G57KD0F00, Filter:Filter_1411-5_1.4x1.1mm, symbol gnss-lib:SAFEB1G57KD0F00
- added J5: SMA_OUT, Connector_Coaxial:SMA_Amphenol_132289_EdgeMount, symbol Connector:Conn_Coaxial
- added R14, R15: 10k, Resistor_SMD:R_0603_1608Metric_Pad0.98x0.95mm_HandSolder, symbol Device:R_Small
- added R16, R20, R23, R26: 249, Resistor_SMD:R_0402_1005Metric, symbol Device:R_Small
- added R17, R18, R19, R21, R22, R24, R25, R27: 61.9, Resistor_SMD:R_0402_1005Metric, symbol Device:R_Small
Connections:
- net GND: now also U5.10 (GND), U5.11 (GND), U5.12 (VSS_EXT/GND), U5.18 (GND), U5.21 (EP/GND), U5.7 (PUP1), U5.8 (PUP2), C28.2, C29.2, C30.2, FL1.2 (GND), FL1.3 (GND), FL1.5 (GND), J5.2 (Ext), R17.1, R18.1, R19.1, R21.1, R22.1, R24.1, R25.1, R27.1
- net GPS_L1_MIX_OUT: now also FL1.1 (IN)
- net at U5.1 (C16): now also R14.2
- net 3V3_MIX: now reaches U5.13 (P/S)
- net 3V3_MIX: now also U5.15 (C8), U5.16 (C4), U5.17 (C2), U5.19 (C1), U5.20 (C0.5), U5.6 (VDD), U5.9 (VDD), C28.1, C29.1, C30.1, R14.1
- net PE4312_RF2: now reaches U5.14 (RF2)
- net PE4312_RF2: now also R19.2, R20.1
- net PE4312_RF1: now reaches U5.2 (RF1)
- net PE4312_RF1: now also R16.2, R18.2
- net at U5.3 (Data): now also R15.2
- net RF_SPI_SCK: now reaches U5.4 (Clock)
- net ATT1_LE: now reaches U5.5 (LE)
- new net: FL1.4 (OUT), R16.1, R17.2
- new net ATT_FIXED_OUT: C31.1, R26.2, R27.2
- new net ATT_FIX_1_OUT: R20.2, R21.2, R22.2, R23.1
- new net ATT_FIX_2_OUT: R23.2, R24.2, R25.2, R26.1
- new net GNSS_RF_OUT: C31.2, J5.1 (In)
- new net RF_SPI_MOSI: R15.1
Other:
- note added: "Конденсаторы C22, C23 расположить у ног VCC LTC5510 C26 общий, максимально к LTC5510"
- note added: "Конденсаторы C28, C29 расположить у ног VDD PE4312 C30 общий, максимально к PE4312"
- moved on the sheet: U5
